Commit message: major change

File: aras_visual_servo_gazebo/robots/aras_visual_servo.URDF (robot description, URDF)
Before this commit: robot aras_visual_servo, 11 links, 10 joints
Links:
- removed link planar_object_2
- link planar_object: mass 1.0 -> 0.3641; geometry collision mesh filename=package://aras_visual_servo_gazebo/meshes/link6.STL; visual mesh filename=package://aras_visual_servo_gazebo/meshes/Part1.STL
Joints:
- removed joint J02
